File: Dossier_kicad/master.kicad_sch (KiCad schematic)
At the start: 7 parts

Commit message: Modifs
Parts:
- removed Batterie1: ~, Library:broche_double, symbol extensions:Broche_Double
- removed ESP32-WROOM-32E1: ~, Library:ESP32_DevKit_38pin_v2, symbol extensions:ESP32WROOM32E
- removed boutton1: ~, Library:broche_tri, symbol extensions:broche_tri
- removed hx711(1)1, hx711(2)1, hx711(3)1, hx711(4)1: ~, Library:TerminalBlock, symbol extensions:broche
Other:
- title: Emetteur -> (none)
